Commit message: Update arm_base.xacro

File: arm/urdf/arm_base.xacro (robot description, xacro)
@@ -51,4 +51,246 @@
         </collision>
     </link>
+    <link name="Link_2">
+        <inertial>
+            <origin xyz="0.00466897689329795 -0.162155529525145 -0.0536740155305947" rpy="0 0 0" />
+            <mass value="2.97373269361303" />
+            <inertia ixx="0.0324167102807371" ixy="0.00297981473551184" ixz="-0.000417973991868469" iyy="0.00996768059711576" iyz="-0.00718854159517085" izz="0.0278574337135304" />
+        </inertial>
+        <visual>
+            <origin xyz="0 0 0" rpy="0 0 0" />
+            <geometry>
+                <mesh filename="file:///home/imbatman/arm_ws/src/arm/meshes/Link_2.STL" />
+            </geometry>
+            <material name="">
+                <color rgba="0.792156862745098 0.819607843137255 0.933333333333333 1" />
+            </material>
+        </visual>
+        <collision>
+            <origin xyz="0 0 0" rpy="0 0 0" />
+            <geometry>
+                <mesh filename="file:///home/imbatman/arm_ws/src/arm/meshes/Link_2.STL" />
+            </geometry>
+        </collision>
+    </link>
+    <link name="Link_3">
+        <inertial>
+            <origin xyz="0.0625571705747566 0.0757694435809385 -0.0197412102243116" rpy="0 0 0" />
+            <mass value="1.45765591046506" />
+            <inertia ixx="0.00668130936621989" ixy="-0.00179290985390331" ixz="0.00110761034441912" iyy="0.00505646179124057" iyz="0.00210611277510792" izz="0.00576711177260289" />
+        </inertial>
+        <visual>
+            <origin xyz="0 0 0" rpy="0 0 0" />
+            <geometry>
+                <mesh filename="file:///home/imbatman/arm_ws/src/arm/meshes/Link_3.STL" />
+            </geometry>
+            <material name="">
+                <color rgba="0.792156862745098 0.819607843137255 0.933333333333333 1" />
+            </material>
+        </visual>
+        <collision>
+            <origin xyz="0 0 0" rpy="0 0 0" />
+            <geometry>
+                <mesh filename="file:///home/imbatman/arm_ws/src/arm/meshes/Link_3.STL" />
+            </geometry>
+        </collision>
+    </link>
+    <link name="Link_4">
+        <inertial>
+            <origin xyz="0.00285172563081149 -0.0260073157026074 0.123071893834179" rpy="0 0 0" />
+            <mass value="0.681236680376837" />
+            <inertia ixx="0.00500336377068867" ixy="2.58053015699419E-05" ixz="-2.97059053335618E-05" iyy="0.00481793578053504" iyz="0.0004000736752812" izz="0.000727383609966516" />
+        </inertial>
+        <visual>
+            <origin xyz="0 0 0" rpy="0 0 0" />
+            <geometry>
+                <mesh filename="file:///home/imbatman/arm_ws/src/arm/meshes/Link_4.STL" />
+            </geometry>
+            <material name="">
+                <color rgba="0.792156862745098 0.819607843137255 0.933333333333333 1" />
+            </material>
+        </visual>
+        <collision>
+            <origin xyz="0 0 0" rpy="0 0 0" />
+            <geometry>
+                <mesh filename="file:///home/imbatman/arm_ws/src/arm/meshes/Link_4.STL" />
+            </geometry>
+        </collision>
+    </link>
+    <link name="Link_5">
+        <inertial>
+            <origin xyz="0.0286748088454602 0.0507749814554782 0.0178696299113226" rpy="0 0 0" />
+            <mass value="0.669420581705739" />
+            <inertia ixx="0.00103371950695079" ixy="-0.000251635215467511" ixz="5.62376905693041E-05" iyy="0.000906027580900811" iyz="0.000124543947445442" izz="0.00143040150433598" />
+        </inertial>
+        <visual>
+            <origin xyz="0 0 0" rpy="0 0 0" />
+            <geometry>
+                <mesh filename="file:///home/imbatman/arm_ws/src/arm/meshes/Link_5.STL" />
+            </geometry>
+            <material name="">
+                <color rgba="1 1 1 1" />
+            </material>
+        </visual>
+        <collision>
+            <origin xyz="0 0 0" rpy="0 0 0" />
+            <geometry>
+                <mesh filename="file:///home/imbatman/arm_ws/src/arm/meshes/Link_5.STL" />
+            </geometry>
+        </collision>
+    </link>
+    <link name="End_effector">
+        <inertial>
+            <origin xyz="1.79542801708177E-05 -0.000122480752124874 0.0096061474499399" rpy="0 0 0" />
+            <mass value="0.0806378641781996" />
+            <inertia ixx="3.24265145588332E-05" ixy="8.12727483201835E-08" ixz="-8.01864845172061E-10" iyy="3.18840006785951E-05" iyz="5.47017248285155E-09" izz="5.90805865629779E-05" />
+        </inertial>
+        <visual>
+            <origin xyz="0 0 0" rpy="0 0 0" />
+            <geometry>
+                <mesh filename="file:///home/imbatman/arm_ws/src/arm/meshes/End_effector.STL" />
+            </geometry>
+            <material name="">
+                <color rgba="0.792156862745098 0.819607843137255 0.933333333333333 1" />
+            </material>
+        </visual>
+        <collision>
+            <origin xyz="0 0 0" rpy="0 0 0" />
+            <geometry>
+                <mesh filename="file:///home/imbatman/arm_ws/src/arm/meshes/End_effector.STL" />
+            </geometry>
+        </collision>
+    </link>
+    <link name="Gripper_base">
+        <inertial>
+            <origin xyz="7.70182675857711E-06 -3.45372920922127E-07 0.0440536598355998" rpy="0 0 0" />
+            <mass value="0.144340160157627" />
+            <inertia ixx="0.00021511317736329" ixy="2.00140097060607E-05" ixz="1.79902238875265E-08" iyy="0.000154298584782079" iyz="-8.00652364350352E-10" izz="0.000101455826246438" />
+        </inertial>
+        <visual>
+            <origin xyz="0 0 0" rpy="0 0 0" />
+            <geometry>
+                <mesh filename="file:///home/imbatman/arm_ws/src/arm/meshes/Gripper_base.STL" />
+            </geometry>
+            <material name="">
+                <color rgba="0.501960784313725 0.501960784313725 0.501960784313725 1" />
+            </material>
+        </visual>
+        <collision>
+            <origin xyz="0 0 0" rpy="0 0 0" />
+            <geometry>
+                <mesh filename="file:///home/imbatman/arm_ws/src/arm/meshes/Gripper_base.STL" />
+            </geometry>
+        </collision>
+    </link>
+    <link name="Gripper_arm_left">
+        <inertial>
+            <origin xyz="0.0415392668558662 0.018365565064578 0.0104837110778671" rpy="0 0 0" />
+            <mass value="0.0127678157416076" />
+            <inertia ixx="1.42841391003646E-06" ixy="-2.11525861803004E-06" ixz="-6.33763992249554E-07" iyy="8.95021294973568E-06" iyz="-3.35016397061264E-07" izz="9.96799180030045E-06" />
+        </inertial>
+        <visual>
+            <origin xyz="0 0 0" rpy="0 0 0" />
+            <geometry>
+                <mesh filename="file:///home/imbatman/arm_ws/src/arm/meshes/Gripper_arm_left.STL" />
+            </geometry>
+            <material name="">
+                <color rgba="1 1 1 1" />
+            </material>
+        </visual>
+        <collision>
+            <origin xyz="0 0 0" rpy="0 0 0" />
+            <geometry>
+                <mesh filename="file:///home/imbatman/arm_ws/src/arm/meshes/Gripper_arm_left.STL" />
+            </geometry>
+        </collision>
+    </link>
+    <link name="left_finger">
+        <inertial>
+            <origin xyz="0.0276961872778643 -0.0147135019401428 0.00437246794423679" rpy="0 0 0" />
+            <mass value="0.0111036375733557" />
+            <inertia ixx="6.4850387494873E-07" ixy="5.06604740618564E-07" ixz="1.51784530404508E-07" iyy="2.82215176126583E-06" iyz="-2.48616489402422E-08" izz="2.89768159875783E-06" />
+        </inertial>
+        <visual>
+            <origin xyz="0 0 0" rpy="0 0 0" />
+            <geometry>
+                <mesh filename="file:///home/imbatman/arm_ws/src/arm/meshes/left_finger.STL" />
+            </geometry>
+            <material name="">
+                <color rgba="0.250980392156863 0.250980392156863 0.250980392156863 1" />
+            </material>
+        </visual>
+        <collision>
+            <origin xyz="0 0 0" rpy="0 0 0" />
+            <geometry>
+                <mesh filename="file:///home/imbatman/arm_ws/src/arm/meshes/left_finger.STL" />
+            </geometry>
+        </collision>
+    </link>
+    <link name="Gripper_arm_right">
+        <inertial>
+            <origin xyz="0.0415392668558654 -0.0183655650645822 -0.0104837110778671" rpy="0 0 0" />
+            <mass value="0.0127678157416076" />
+            <inertia ixx="1.42841391003647E-06" ixy="2.11525861803006E-06" ixz="6.33763992249559E-07" iyy="8.95021294973568E-06" iyz="-3.35016397061264E-07" izz="9.96799180030045E-06" />
+        </inertial>
+        <visual>
+            <origin xyz="0 0 0" rpy="0 0 0" />
+            <geometry>
+                <mesh filename="file:///home/imbatman/arm_ws/src/arm/meshes/Gripper_arm_right.STL" />
+            </geometry>
+            <material name="">
+                <color rgba="1 1 1 1" />
+            </material>
+        </visual>
+        <collision>
+            <origin xyz="0 0 0" rpy="0 0 0" />
+            <geometry>
+                <mesh filename="file:///home/imbatman/arm_ws/src/arm/meshes/Gripper_arm_right.STL" />
+            </geometry>
+        </collision>
+    </link>
+    <link name="Right_finger">
+        <inertial>
+            <origin xyz="0.027616145582933 0.0148633586436651 -0.00432757204095563" rpy="0 0 0" />
+            <mass value="0.0111036338959234" />
+            <inertia ixx="6.54555696498015E-07" ixy="-5.18309449389992E-07" ixz="-1.5529184263656E-07" iyy="2.81659729446906E-06" iyz="-2.65257515723312E-08" izz="2.8971822175015E-06" />
+        </inertial>
+        <visual>
+            <origin xyz="0 0 0" rpy="0 0 0" />
+            <geometry>
+                <mesh filename="file:///home/imbatman/arm_ws/src/arm/meshes/Right_finger.STL" />
+            </geometry>
+            <material name="">
+                <color rgba="0.250980392156863 0.250980392156863 0.250980392156863 1" />
+            </material>
+        </visual>
+        <collision>
+            <origin xyz="0 0 0" rpy="0 0 0" />
+            <geometry>
+                <mesh filename="file:///home/imbatman/arm_ws/src/arm/meshes/Right_finger.STL" />
+            </geometry>
+        </collision>
+    </link>
+    <link name="RGB_camera">
+        <inertial>
+            <origin xyz="0.00952416675236908 0.000322242755626256 -0.0086020702736585" rpy="0 0 0" />
+            <mass value="0.00851529124922691" />
+            <inertia ixx="5.72032823016266E-07" ixy="-1.40620704134015E-22" ixz="3.97046694025453E-22" iyy="5.72032823016266E-07" iyz="-2.64697796016969E-23" izz="8.87510252850143E-07" />
+        </inertial>
+        <visual>
+            <origin xyz="0 0 0" rpy="0 0 0" />
+            <geometry>
+                <mesh filename="file:///home/imbatman/arm_ws/src/arm/meshes/RGB_camera.STL" />
+            </geometry>
+            <material name="">
+                <color rgba="0.792156862745098 0.819607843137255 0.933333333333333 1" />
+            </material>
+        </visual>
+        <collision>
+            <origin xyz="0 0 0" rpy="0 0 0" />
+            <geometry>
+                <mesh filename="file:///home/imbatman/arm_ws/src/arm/meshes/RGB_camera.STL" />
+            </geometry>
+        </collision>
+    </link>
     <joint name="Joint_1" type="revolute">
         <origin xyz="0 0 0.154" rpy="0 0 -1.5707963267949" />
@@ -58,26 +300,4 @@
         <limit lower="0" upper="6.28" effort="11" velocity="2" />
     </joint>
-    <link name="Link_2">
-        <inertial>
-            <origin xyz="0.00466897689329795 -0.162155529525145 -0.0536740155305947" rpy="0 0 0" />
-            <mass value="2.97373269361303" />
-            <inertia ixx="0.0324167102807371" ixy="0.00297981473551184" ixz="-0.000417973991868469" iyy="0.00996768059711576" iyz="-0.00718854159517085" izz="0.0278574337135304" />
-        </inertial>
-        <visual>
-            <origin xyz="0 0 0" rpy="0 0 0" />
-            <geometry>
-                <mesh filename="file:///home/imbatman/arm_ws/src/arm/meshes/Link_2.STL" />
-            </geometry>
-            <material name="">
-                <color rgba="0.792156862745098 0.819607843137255 0.933333333333333 1" />
-            </material>
-        </visual>
-        <collision>
-            <origin xyz="0 0 0" rpy="0 0 0" />
-            <geometry>
-                <mesh filename="file:///home/imbatman/arm_ws/src/arm/meshes/Link_2.STL" />
-            </geometry>
-        </collision>
-    </link>
     <joint name="Joint_2" type="revolute">
         <origin xyz="-0.0650932810459635 0.00632651267849924 0.115" rpy="-1.5707963267949 0 1.5707963267949" />
@@ -87,26 +307,4 @@
         <limit lower="0" upper="2.059" effort="11" velocity="2" />
     </joint>
-    <link name="Link_3">
-        <inertial>
-            <origin xyz="0.0625571705747566 0.0757694435809385 -0.0197412102243116" rpy="0 0 0" />
-            <mass value="1.45765591046506" />
-            <inertia ixx="0.00668130936621989" ixy="-0.00179290985390331" ixz="0.00110761034441912" iyy="0.00505646179124057" iyz="0.00210611277510792" izz="0.00576711177260289" />
-        </inertial>
-        <visual>
-            <origin xyz="0 0 0" rpy="0 0 0" />
-            <geometry>
-                <mesh filename="file:///home/imbatman/arm_ws/src/arm/meshes/Link_3.STL" />
-            </geometry>
-            <material name="">
-                <color rgba="0.792156862745098 0.819607843137255 0.933333333333333 1" />
-            </material>
-        </visual>
-        <collision>
-            <origin xyz="0 0 0" rpy="0 0 0" />
-            <geometry>
-                <mesh filename="file:///home/imbatman/arm_ws/src/arm/meshes/Link_3.STL" />
-            </geometry>
-        </collision>
-    </link>
     <joint name="Joint_3" type="revolute">
         <origin xyz="0.0530599818434298 -0.28455 -0.00515697845398792" rpy="0 0 0" />
@@ -116,26 +314,4 @@
         <limit lower="0" upper="3.8" effort="11" velocity="2" />
     </joint>
-    <link name="Link_4">
-        <inertial>
-            <origin xyz="0.00285172563081149 -0.0260073157026074 0.123071893834179" rpy="0 0 0" />
-            <mass value="0.681236680376837" />
-            <inertia ixx="0.00500336377068867" ixy="2.58053015699419E-05" ixz="-2.97059053335618E-05" iyy="0.00481793578053504" iyz="0.0004000736752812" izz="0.000727383609966516" />
-        </inertial>
-        <visual>
-            <origin xyz="0 0 0" rpy="0 0 0" />
-            <geometry>
-                <mesh filename="file:///home/imbatman/arm_ws/src/arm/meshes/Link_4.STL" />
-            </geometry>
-            <material name="">
-                <color rgba="0.792156862745098 0.819607843137255 0.933333333333333 1" />
-            </material>
-        </visual>
-        <collision>
-            <origin xyz="0 0 0" rpy="0 0 0" />
-            <geometry>
-                <mesh filename="file:///home/imbatman/arm_ws/src/arm/meshes/Link_4.STL" />
-            </geometry>
-        </collision>
-    </link>
     <joint name="Joint_4" type="revolute">
         <origin xyz="0.0784902400245383 0.17127 -0.0648971665089489" rpy="-1.5707963267949 0 0" />
@@ -145,26 +321,4 @@
         <limit lower="0" upper="6.28" effort="11" velocity="2" />
     </joint>
-    <link name="Link_5">
-        <inertial>
-            <origin xyz="0.0286748088454602 0.0507749814554782 0.0178696299113226" rpy="0 0 0" />
-            <mass value="0.669420581705739" />
-            <inertia ixx="0.00103371950695079" ixy="-0.000251635215467511" ixz="5.62376905693041E-05" iyy="0.000906027580900811" iyz="0.000124543947445442" izz="0.00143040150433598" />
-        </inertial>
-        <visual>
-            <origin xyz="0 0 0" rpy="0 0 0" />
-            <geometry>
-                <mesh filename="file:///home/imbatman/arm_ws/src/arm/meshes/Link_5.STL" />
-            </geometry>
-            <material name="">
-                <color rgba="1 1 1 1" />
-            </material>
-        </visual>
-        <collision>
-            <origin xyz="0 0 0" rpy="0 0 0" />
-            <geometry>
-                <mesh filename="file:///home/imbatman/arm_ws/src/arm/meshes/Link_5.STL" />
-            </geometry>
-        </collision>
-    </link>
     <joint name="Joint_5" type="revolute">
         <origin xyz="-0.000337607480855595 0.00347363227600019 0.2" rpy="-1.5707963267949 0 0" />
@@ -174,26 +328,4 @@
         <limit lower="-0.83" upper="2.9" effort="11" velocity="2" />
     </joint>
-    <link name="End_effector">
-        <inertial>
-            <origin xyz="1.79542801708177E-05 -0.000122480752124874 0.0096061474499399" rpy="0 0 0" />
-            <mass value="0.0806378641781996" />
-            <inertia ixx="3.24265145588332E-05" ixy="8.12727483201835E-08" ixz="-8.01864845172061E-10" iyy="3.18840006785951E-05" iyz="5.47017248285155E-09" izz="5.90805865629779E-05" />
-        </inertial>
-        <visual>
-            <origin xyz="0 0 0" rpy="0 0 0" />
-            <geometry>
-                <mesh filename="file:///home/imbatman/arm_ws/src/arm/meshes/End_effector.STL" />
-            </geometry>
-            <material name="">
-                <color rgba="0.792156862745098 0.819607843137255 0.933333333333333 1" />
-            </material>
-        </visual>
-        <collision>
-            <origin xyz="0 0 0" rpy="0 0 0" />
-            <geometry>
-                <mesh filename="file:///home/imbatman/arm_ws/src/arm/meshes/End_effector.STL" />
-            </geometry>
-        </collision>
-    </link>
     <joint name="End_effector_Joint" type="revolute">
         <origin xyz="0.0872672717341501 0.0490789751008787 0.0185287556820571" rpy="1.47993501318796 -0.0336819095690923 1.21676367586924" />
@@ -203,26 +335,4 @@
         <limit lower="0" upper="6.28" effort="11" velocity="2" />
     </joint>
-    <link name="Gripper_base">
-        <inertial>
-            <origin xyz="7.70182675857711E-06 -3.45372920922127E-07 0.0440536598355998" rpy="0 0 0" />
-            <mass value="0.144340160157627" />
-            <inertia ixx="0.00021511317736329" ixy="2.00140097060607E-05" ixz="1.79902238875265E-08" iyy="0.000154298584782079" iyz="-8.00652364350352E-10" izz="0.000101455826246438" />
-        </inertial>
-        <visual>
-            <origin xyz="0 0 0" rpy="0 0 0" />
-            <geometry>
-                <mesh filename="file:///home/imbatman/arm_ws/src/arm/meshes/Gripper_base.STL" />
-            </geometry>
-            <material name="">
-                <color rgba="0.501960784313725 0.501960784313725 0.501960784313725 1" />
-            </material>
-        </visual>
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