Commit message: Update arm.urdf

File: arm/urdf/arm.urdf (robot description, URDF)
Before this commit: robot arm, 14 links, 13 joints
Links:
- link End_effector: geometry collision mesh filename=file:///home/imbatman/arm_ws/src/arm/meshes/End_effector.STL; visual mesh filename=file:///home/imbatman/arm_ws/src/arm/meshes/End_effector.STL
- link Gripper_arm_left: geometry collision mesh filename=file:///home/imbatman/arm_ws/src/arm/meshes/Gripper_arm_lef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; visual mesh filename=file:///home/imbatman/arm_ws/src/arm/meshes/Gripper_arm_lef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
- link Gripper_arm_right: geometry collision mesh filename=file:///home/imbatman/arm_ws/src/arm/meshes/Gripper_arm_rig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; visual mesh filename=file:///home/imbatman/arm_ws/src/arm/meshes/Gripper_arm_rig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
- link Gripper_base: geometry collision mesh filename=file:///home/imbatman/arm_ws/src/arm/meshes/Gripper_base.STL; visual mesh filename=file:///home/imbatman/arm_ws/src/arm/meshes/Gripper_base.STL
- link Link_1: geometry collision mesh filename=file:///home/imbatman/arm_ws/src/arm/meshes/Link_1.STL; visual mesh filename=file:///home/imbatman/arm_ws/src/arm/meshes/Link_1.STL
- link Link_2: geometry collision mesh filename=file:///home/imbatman/arm_ws/src/arm/meshes/Link_2.STL; visual mesh filename=file:///home/imbatman/arm_ws/src/arm/meshes/Link_2.STL
- link Link_3: geometry collision mesh filename=file:///home/imbatman/arm_ws/src/arm/meshes/Link_3.STL; visual mesh filename=file:///home/imbatman/arm_ws/src/arm/meshes/Link_3.STL
- link Link_4: geometry collision mesh filename=file:///home/imbatman/arm_ws/src/arm/meshes/Link_4.STL; visual mesh filename=file:///home/imbatman/arm_ws/src/arm/meshes/Link_4.STL
- link Link_5: geometry collision mesh filename=file:///home/imbatman/arm_ws/src/arm/meshes/Link_5.STL; visual mesh filename=file:///home/imbatman/arm_ws/src/arm/meshes/Link_5.STL
- link RGB_camera: geometry collision mesh filename=file:///home/imbatman/arm_ws/src/arm/meshes/RGB_camera.STL; visual mesh filename=file:///home/imbatman/arm_ws/src/arm/meshes/RGB_camera.STL
- link Right_finger: geometry collision mesh filename=file:///home/imbatman/arm_ws/src/arm/meshes/Right_finger.STL; visual mesh filename=file:///home/imbatman/arm_ws/src/arm/meshes/Right_finger.STL
- link arm_base_link: geometry collision mesh filename=file:///home/imbatman/arm_ws/src/arm/meshes/arm_base_link.S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; visual mesh filename=file:///home/imbatman/arm_ws/src/arm/meshes/arm_base_link.S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
- link left_finger: geometry collision mesh filename=file:///home/imbatman/arm_ws/src/arm/meshes/left_finger.STL; visual mesh filename=file:///home/imbatman/arm_ws/src/arm/meshes/left_finger.STL
Joints:
- joint Gripper_arm_right_Joint: limit lower=0 upper=0 effort=11 velocity=2 -> lower=-1.22 upper=0.06 effort=11 velocity=2
