Commit message: Update arm_gazebo.xacro

File: arm/urdf/arm_gazebo.xacro (robot description, xacro)
@@ -21,3 +21,50 @@
     </sensor>
   </gazebo>
+  <gazebo reference="arm_base_link">
+        <material>Gazebo/LightGrey</material>
+    </gazebo>
+    <!-- Gazebo material for Link_1 -->
+    <gazebo reference="Link_1">
+        <material>Gazebo/Blue</material>
+    </gazebo>
+    <!-- Gazebo material for Link_2 -->
+    <gazebo reference="Link_2">
+        <material>Gazebo/Blue</material>
+    </gazebo>
+    <!-- Gazebo material for Link_3 -->
+    <gazebo reference="Link_3">
+        <material>Gazebo/Blue</material>
+    </gazebo>
+    <!-- Gazebo material for Link_4 -->
+    <gazebo reference="Link_4">
+        <material>Gazebo/Blue</material>
+    </gazebo>
+    <!-- Gazebo material for Link_5 -->
+    <gazebo reference="Link_5">
+        <material>Gazebo/White</material>
+    </gazebo>
+    <!-- Gazebo material for End_effector -->
+    <gazebo reference="End_effector">
+        <material>Gazebo/Blue</material>
+    </gazebo>
+    <!-- Gazebo material for Gripper_base -->
+    <gazebo reference="Gripper_base">
+        <material>Gazebo/Grey</material>
+    </gazebo>
+    <!-- Gazebo material for Gripper_arm_left -->
+    <gazebo reference="Gripper_arm_left">
+        <material>Gazebo/White</material>
+    </gazebo>
+    <!-- Gazebo material for left_finger -->
+    <gazebo reference="left_finger">
+        <material>Gazebo/DarkGrey</material>
+    </gazebo>
+    <!-- Gazebo material for Gripper_arm_right -->
+    <gazebo reference="Gripper_arm_right">
+        <material>Gazebo/White</material>
+    </gazebo>
+    <!-- Gazebo material for Right_finger -->
+    <gazebo reference="Right_finger">
+        <material>Gazebo/DarkGrey</material>
+    </gazebo>
 </robot>
